File: CAD/eurocard mux.kicad_pcb (KiCad board)
At the start: 4 copper layers, 160 x 100 mm, 71 parts, among them J1 Conn_01x16, J2 Conn_01x16, J3 1847712, K1 AGQ200S12Z, K10 AGQ200S12Z, K11 AGQ200S12Z, K12 AGQ200S12Z, K13 AGQ200S12Z, K14 AGQ200S12Z, K15 AGQ200S12Z, K16 AGQ200S12Z, K17 AGQ200S12Z, K18 AGQ200S12Z, K19 AGQ200S12Z, K2 AGQ200S12Z, K20 AGQ200S12Z, K21 AGQ200S12Z, K22 AGQ200S12Z, K23 AGQ200S12Z, K24 AGQ200S12Z, K25 AGQ200S12Z, K26 AGQ200S12Z, K27 AGQ200S12Z, K28 AGQ200S12Z, K29 AGQ200S12Z, K3 AGQ200S12Z, K30 AGQ200S12Z, K31 AGQ200S12Z, K32 AGQ200S12Z, K33 AGQ200S12Z, K34 AGQ200S12Z, K35 AGQ200S12Z, K36 AGQ200S12Z, K37 AGQ200S12Z, K38 AGQ200S12Z, K39 AGQ200S12Z, K4 AGQ200S12Z, K40 AGQ200S12Z, K41 AGQ200S12Z, K42 AGQ200S12Z, K43 AGQ200S12Z, K44 AGQ200S12Z, K45 AGQ200S12Z, K46 AGQ200S12Z, K47 AGQ200S12Z, K48 AGQ200S12Z, K5 AGQ200S12Z, K6 AGQ200S12Z, K7 AGQ200S12Z, K8 AGQ200S12Z, K9 AGQ200S12Z, U1 SN74LVC3G34DCUR, U2 SN74LVC3G34DCUR, U3 TPIC6C596, U4 TPIC6C596, U5 TPIC6C596, U6 TPIC6C596, U7 TPIC6C596, U8 TPIC6C596

Commit message: Feat: WIP
Parts:
- added C10: 0.1uF, Diode_SMD:D_0603_1608Metric, F.Cu at (148.8, 136.1)
- added C11: 0.1uF, Diode_SMD:D_0603_1608Metric, F.Cu at (159.8, 136.1)
- added C12: 0.1uF, Diode_SMD:D_0603_1608Metric, F.Cu at (170.8, 136.1)
- added C13: 0.1uF, Diode_SMD:D_0603_1608Metric, F.Cu at (181.8, 136.1)
- added C14: 0.1uF, Diode_SMD:D_0603_1608Metric, F.Cu at (192.8, 136.1)
- added C9: 0.1uF, Diode_SMD:D_0603_1608Metric, F.Cu at (137.8, 136.1)
- added J4: 1847712, Connector_Phoenix_MC_HighVoltage:PhoenixContact_MC_1,5_12-GF-5.08_1x12_P5.08mm_Horizontal_ThreadedFlange_MountHole, F.Cu at (198.9, 91.0)
- added K49: AGQ200S12Z, muxlib_footprints:Relay_2P2T_10x6mm_TE_IMxxG, F.Cu at (141.0, 99.0)
- added K50: AGQ200S12Z, muxlib_footprints:Relay_2P2T_10x6mm_TE_IMxxG, F.Cu at (141.0, 108.0)
- added K51: AGQ200S12Z, muxlib_footprints:Relay_2P2T_10x6mm_TE_IMxxG, F.Cu at (141.0, 117.0)
- added K52: AGQ200S12Z, muxlib_footprints:Relay_2P2T_10x6mm_TE_IMxxG, F.Cu at (141.0, 126.0)
- added K53: AGQ200S12Z, muxlib_footprints:Relay_2P2T_10x6mm_TE_IMxxG, B.Cu at (141.0, 99.0)
- added K54: AGQ200S12Z, muxlib_footprints:Relay_2P2T_10x6mm_TE_IMxxG, B.Cu at (141.0, 108.0)
- added K55: AGQ200S12Z, muxlib_footprints:Relay_2P2T_10x6mm_TE_IMxxG, B.Cu at (141.0, 117.0)
- added K56: AGQ200S12Z, muxlib_footprints:Relay_2P2T_10x6mm_TE_IMxxG, B.Cu at (141.0, 126.0)
- added K57: AGQ200S12Z, muxlib_footprints:Relay_2P2T_10x6mm_TE_IMxxG, F.Cu at (152.0, 99.0)
- added K58: AGQ200S12Z, muxlib_footprints:Relay_2P2T_10x6mm_TE_IMxxG, F.Cu at (152.0, 108.0)
- added K59: AGQ200S12Z, muxlib_footprints:Relay_2P2T_10x6mm_TE_IMxxG, F.Cu at (152.0, 117.0)
- added K60: AGQ200S12Z, muxlib_footprints:Relay_2P2T_10x6mm_TE_IMxxG, F.Cu at (152.0, 126.0)
- added K61: AGQ200S12Z, muxlib_footprints:Relay_2P2T_10x6mm_TE_IMxxG, B.Cu at (152.0, 99.0)
- added K62: AGQ200S12Z, muxlib_footprints:Relay_2P2T_10x6mm_TE_IMxxG, B.Cu at (152.0, 108.0)
- added K63: AGQ200S12Z, muxlib_footprints:Relay_2P2T_10x6mm_TE_IMxxG, B.Cu at (152.0, 117.0)
- added K64: AGQ200S12Z, muxlib_footprints:Relay_2P2T_10x6mm_TE_IMxxG, B.Cu at (152.0, 126.0)
- added K65: AGQ200S12Z, muxlib_footprints:Relay_2P2T_10x6mm_TE_IMxxG, F.Cu at (163.0, 99.0)
- added K66: AGQ200S12Z, muxlib_footprints:Relay_2P2T_10x6mm_TE_IMxxG, F.Cu at (163.0, 108.0)
- added K67: AGQ200S12Z, muxlib_footprints:Relay_2P2T_10x6mm_TE_IMxxG, F.Cu at (163.0, 117.0)
- added K68: AGQ200S12Z, muxlib_footprints:Relay_2P2T_10x6mm_TE_IMxxG, F.Cu at (163.0, 126.0)
- added K69: AGQ200S12Z, muxlib_footprints:Relay_2P2T_10x6mm_TE_IMxxG, B.Cu at (163.0, 99.0)
- added K70: AGQ200S12Z, muxlib_footprints:Relay_2P2T_10x6mm_TE_IMxxG, B.Cu at (163.0, 108.0)
- added K71: AGQ200S12Z, muxlib_footprints:Relay_2P2T_10x6mm_TE_IMxxG, B.Cu at (163.0, 117.0)
- added K72: AGQ200S12Z, muxlib_footprints:Relay_2P2T_10x6mm_TE_IMxxG, B.Cu at (163.0, 126.0)
- added K73: AGQ200S12Z, muxlib_footprints:Relay_2P2T_10x6mm_TE_IMxxG, F.Cu at (174.0, 99.0)
- added K74: AGQ200S12Z, muxlib_footprints:Relay_2P2T_10x6mm_TE_IMxxG, F.Cu at (174.0, 108.0)
- added K75: AGQ200S12Z, muxlib_footprints:Relay_2P2T_10x6mm_TE_IMxxG, F.Cu at (174.0, 117.0)
- added K76: AGQ200S12Z, muxlib_footprints:Relay_2P2T_10x6mm_TE_IMxxG, F.Cu at (174.0, 126.0)
- added K77: AGQ200S12Z, muxlib_footprints:Relay_2P2T_10x6mm_TE_IMxxG, B.Cu at (174.0, 99.0)
- added K78: AGQ200S12Z, muxlib_footprints:Relay_2P2T_10x6mm_TE_IMxxG, B.Cu at (174.0, 108.0)
- added K79: AGQ200S12Z, muxlib_footprints:Relay_2P2T_10x6mm_TE_IMxxG, B.Cu at (174.0, 117.0)
- added K80: AGQ200S12Z, muxlib_footprints:Relay_2P2T_10x6mm_TE_IMxxG, B.Cu at (174.0, 126.0)
- added K81: AGQ200S12Z, muxlib_footprints:Relay_2P2T_10x6mm_TE_IMxxG, F.Cu at (185.0, 99.0)
- added K82: AGQ200S12Z, muxlib_footprints:Relay_2P2T_10x6mm_TE_IMxxG, F.Cu at (185.0, 108.0)
- added K83: AGQ200S12Z, muxlib_footprints:Relay_2P2T_10x6mm_TE_IMxxG, F.Cu at (185.0, 117.0)
- added K84: AGQ200S12Z, muxlib_footprints:Relay_2P2T_10x6mm_TE_IMxxG, F.Cu at (185.0, 126.0)
- added K85: AGQ200S12Z, muxlib_footprints:Relay_2P2T_10x6mm_TE_IMxxG, B.Cu at (185.0, 99.0)
- added K86: AGQ200S12Z, muxlib_footprints:Relay_2P2T_10x6mm_TE_IMxxG, B.Cu at (185.0, 108.0)
- added K87: AGQ200S12Z, muxlib_footprints:Relay_2P2T_10x6mm_TE_IMxxG, B.Cu at (185.0, 117.0)
- added K88: AGQ200S12Z, muxlib_footprints:Relay_2P2T_10x6mm_TE_IMxxG, B.Cu at (185.0, 126.0)
- added K89: AGQ200S12Z, muxlib_footprints:Relay_2P2T_10x6mm_TE_IMxxG, F.Cu at (196.0, 99.0)
- added K90: AGQ200S12Z, muxlib_footprints:Relay_2P2T_10x6mm_TE_IMxxG, F.Cu at (196.0, 108.0)
- added K91: AGQ200S12Z, muxlib_footprints:Relay_2P2T_10x6mm_TE_IMxxG, F.Cu at (196.0, 117.0)
- added K92: AGQ200S12Z, muxlib_footprints:Relay_2P2T_10x6mm_TE_IMxxG, F.Cu at (196.0, 126.0)
- added K93: AGQ200S12Z, muxlib_footprints:Relay_2P2T_10x6mm_TE_IMxxG, B.Cu at (196.0, 99.0)
- added K94: AGQ200S12Z, muxlib_footprints:Relay_2P2T_10x6mm_TE_IMxxG, B.Cu at (196.0, 108.0)
- added K95: AGQ200S12Z, muxlib_footprints:Relay_2P2T_10x6mm_TE_IMxxG, B.Cu at (196.0, 117.0)
- added K96: AGQ200S12Z, muxlib_footprints:Relay_2P2T_10x6mm_TE_IMxxG, B.Cu at (196.0, 126.0)
- added U10: TPIC6C596, Package_SO:TSSOP-16_4.4x5mm_P0.65mm, F.Cu at (152.6, 136.4)
- added U11: TPIC6C596, Package_SO:TSSOP-16_4.4x5mm_P0.65mm, F.Cu at (163.6, 136.4)
- added U12: TPIC6C596, Package_SO:TSSOP-16_4.4x5mm_P0.65mm, F.Cu at (174.6, 136.4)
- added U13: TPIC6C596, Package_SO:TSSOP-16_4.4x5mm_P0.65mm, F.Cu at (185.6, 136.4)
- added U14: TPIC6C596, Package_SO:TSSOP-16_4.4x5mm_P0.65mm, F.Cu at (196.6, 136.4)
- added U9: TPIC6C596, Package_SO:TSSOP-16_4.4x5mm_P0.65mm, F.Cu at (141.6, 136.4)
- J1: footprint Connector_IDC:IDC-Header_2x08_P2.54mm_Vertical -> Connector_IDC:IDC-Header_2x08_P2.54mm_Horizontal; moved to B.Cu
- J2: footprint Connector_IDC:IDC-Header_2x08_P2.54mm_Vertical -> Connector_IDC:IDC-Header_2x08_P2.54mm_Horizontal
- K13, K14, K15, K16, K21, K22, K23, K24, K29, K30, K31, K32, K37, K38, K39, K40, K45, K46, K47, K48, K5, K6, K7, K8: moved to B.Cu
- moved U1 186.2 mm to (202.0, 139.0), turned to 90 degrees
- moved U2 178.9 mm to (202.0, 133.0), turned to 90 degrees
- moved C1 167.9 mm to (235.3, 136.2)
- moved C2 167.9 mm to (235.3, 138.8)
- moved K48 63.0 mm to (130.0, 126.0)
- moved K45 63.0 mm to (130.0, 99.0)
- moved K46 63.0 mm to (130.0, 108.0)
- moved K47 63.0 mm to (130.0, 117.0)
- moved C8 52.0 mm to (126.8, 136.1)
- moved K40 52.0 mm to (119.0, 126.0)
- moved K41 52.0 mm to (130.0, 99.0)
- moved K42 52.0 mm to (130.0, 108.0)
- moved K43 52.0 mm to (130.0, 117.0)
- moved K44 52.0 mm to (130.0, 126.0)
- moved U8 52.0 mm to (130.6, 136.4)
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Routing:
- net +12V: track 351.2 -> 702.4 mm, vias 12 -> 24
- net OUT_N: track 43.3 -> 107.4 mm
- net Net-(U9-DRAIN3): track 0.00 -> 44.3 mm, vias 0 -> 1
- net Net-(U14-DRAIN3): track 0.00 -> 44.3 mm, vias 0 -> 1
- net Net-(U13-DRAIN3): track 0.00 -> 44.3 mm, vias 0 -> 1
- net Net-(U12-DRAIN3): track 0.00 -> 44.3 mm, vias 0 -> 1
- net Net-(U11-DRAIN3): track 0.00 -> 44.3 mm, vias 0 -> 1
- net Net-(U10-DRAIN3): track 0.00 -> 44.3 mm, vias 0 -> 1
- net Net-(U9-DRAIN2): track 0.00 -> 36.7 mm, vias 0 -> 1
- net Net-(U14-DRAIN2): track 0.00 -> 36.7 mm, vias 0 -> 1
- net Net-(U13-DRAIN2): track 0.00 -> 36.7 mm, vias 0 -> 1
- net Net-(U12-DRAIN2): track 0.00 -> 36.7 mm, vias 0 -> 1
- net Net-(U11-DRAIN2): track 0.00 -> 36.7 mm, vias 0 -> 1
- net Net-(U10-DRAIN2): track 0.00 -> 36.7 mm, vias 0 -> 1
- net CH_1: track 46.0 -> 11.8 mm
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
Commit message: Feat:WIP push
Parts:
- added J5: Conn_01x02, Connector_Phoenix_MC_HighVoltage:PhoenixContact_MC_1,5_2-G-5.08_1x02_P5.08mm_Horizontal, B.Cu at (210.1, 97.9)
- added J6: Conn_01x02, Connector_Phoenix_MC_HighVoltage:PhoenixContact_MC_1,5_2-G-5.08_1x02_P5.08mm_Horizontal, F.Cu at (59.9, 97.5)
- added JP1: Jumper_2_Bridged, Resistor_SMD:R_0805_2012Metric, F.Cu at (65.0, 108.0)
- added JP2: Jumper_2_Bridged, Resistor_SMD:R_0805_2012Metric, F.Cu at (62.0, 107.9)
- added JP3: Jumper_2_Bridged, Resistor_SMD:R_0805_2012Metric, F.Cu at (204.0, 108.0)
- added JP4: Jumper_2_Bridged, Resistor_SMD:R_0805_2012Metric, F.Cu at (208.0, 108.0)
Connections:
- J1 pad 15: OUT_P -> Net-(J1-Pin_15)
- J1 pad 16: OUT_N -> Net-(J1-Pin_16)
- J2 pad 1: +5V -> serial_return
- J2 pad 10: ch2 -> +5V
- J2 pad 12: ch4 -> ch1
- J2 pad 15: OUT_P -> Net-(J2-Pin_15)
- J2 pad 16: OUT_N -> Net-(J2-Pin_16)
- J2 pad 2: +12V -> serial_in
- J2 pad 3: serial_return -> serial_clock
- J2 pad 4: serial_in -> transfer
- J2 pad 5: serial_clock -> synchronous_clear
- J2 pad 6: transfer -> device_enable
- J2 pad 7: synchronous_clear -> ch2
- J2 pad 8: device_enable -> ch4
- J2 pad 9: ch1 -> +12V
Routing:
- net OUT_N: track 107.4 -> 294.1 mm
- net OUT_P: track 44.4 -> 217.0 mm
- net ch4: track 41.2 -> 184.4 mm
- net ch1: track 48.4 -> 190.2 mm
- net +12V: track 702.4 -> 842.8 mm
- net ch2: track 41.4 -> 180.6 mm
- net ch3: track 46.9 -> 185.5 mm
- net device_enable: track 10.3 -> 131.7 mm
- net transfer: track 33.2 -> 154.2 mm
- net serial_clock: track 30.3 -> 151.3 mm
- net +5V: track 35.6 -> 156.6 mm
- net Net-(J1-Pin_15): track 0.00 -> 5.57 mm
- net Net-(J1-Pin_16): track 0.00 -> 4.96 mm
- net Net-(J2-Pin_15): track 0.00 -> 4.74 mm
- net Net-(J2-Pin_16): track 0.00 -> 4.63 mm
