File: CAD/Relay_group.kicad_sch (KiCad schematic)
At the start: 10 parts, among them K1 AGQ200S12Z, K2 AGQ200S12Z, K3 AGQ200S12Z, K4 AGQ200S12Z, K5 AGQ200S12Z, K6 AGQ200S12Z, K7 AGQ200S12Z, K8 AGQ200S12Z, U3 TPIC6C596

Commit message: New formfactor and remake
Parts:
- C3: footprint Diode_SMD:D_0603_1608Metric -> Capacitor_SMD:C_0603_1608Metric; Digikey CL10B104KB8NFNC -> (none); LCSC Part # CL10B104KB8NFNC -> (none); MPN (none) -> 0603 100nF 24v
- K1, K2, K3, K4, K5, K6, K7, K8: Digikey AGQ200S12Z -> (none); LCSC Part # AGQ200S12Z -> (none); MPN (none) -> AGQ200S12Z
- U3: Digikey TPIC6C596PWR -> (none); LCSC Part # TPIC6C596PWR -> (none); MPN (none) -> TPIC6C596PWR
Connections:
- net A_CH2_CH4: now reaches K4.8, U3.11 (DRAIN4)
- net A_CH1_CH3: now reaches K3.8, U3.12 (DRAIN5)
- net A_CHANNEL_X_POLARITY: now reaches K2.8, U3.13 (DRAIN6)
- net A_SAMPLE_INJECT: now reaches K1.8, U3.14 (DRAIN7)
- net B_CH2_CH4: now reaches K8.8, U3.3 (DRAIN0)
- net B_CH1_CH3: now reaches K7.8, U3.4 (DRAIN1)
- net B_CHANNEL_X_POLARITY: now reaches K6.8, U3.5 (DRAIN2)
- net B_SAMPLE_INJECT: now reaches K5.8, U3.6 (DRAIN3)
Other:
- note added: "CH1,2,3,4/OUTN,P"
- note added: "CH1/CH3"
- note added: "CH2/CH4"
- note added: "SAMPLE/INJECT"
