File: CAD/buffer.kicad_sch (KiCad schematic)
At the start: 4 parts, among them U1 SN74LVC3G34DCUR, U2 SN74LVC3G34DCUR

Commit message: New formfactor and remake
Parts:
- C1, C2: footprint Diode_SMD:D_0603_1608Metric -> Capacitor_SMD:C_0603_1608Metric; Digikey CL10B104KB8NFNC -> (none); LCSC Part # CL10B104KB8NFNC -> (none); MPN (none) -> 0603 100nF 24v
- U1, U2: Digikey SN74LVC3G34DCUR -> (none); LCSC Part # SN74LVC3G34DCUR -> (none); MPN (none) -> SN74LVC3G34DCUR
